File: StepperNode_Gimbal_420ma.sch (KiCad schematic (older format))
At the start: 0 parts

Commit message: Update gimbal and brake MLP position sensor interfaces
Parts:
- added C? (x4): 100nF, symbol C
- added C? (x4): 1uF, symbol C
- added D? (x4): 1N4148, symbol D
- added P?: CONN_01X08_2MNT, symbol CONN_01X08_2MNT
- added U? (x4): RCV420JP, symbol RCV420JP
Connections:
- net labels added: +24V_A, GIMBAL_MLP1_420MA, GIMBAL_MLP2_420MA, GIMBAL_MLP3_420MA, GNDA
- net labels removed: GIMBAL4_MLP
- wire segments 0 -> 40
Other:
- note added: "Interface to MLP's\nOn the gimbals"
- note added: "Original Author: SafetyLok"
- note added: "rLoop - Stepper Node\nGimbal MLP 4-20 Interface\n"
