File: elec-stepper-node.sch (KiCad schematic (older format))
At the start: 29 parts

Commit message: Remove Gimbal Functions
Connections:
- net labels added: A_BRAKE1_DIR, A_BRAKE1_STEP, A_BRAKE2_DIR, A_BRAKE2_STEP, BRAKE1_DIR, BRAKE1_STEP, BRAKE2_DIR, BRAKE2_STEP, B_BRAKE1_DIR, B_BRAKE1_STEP, B_BRAKE2_DIR, B_BRAKE2_STEP
- net labels removed: A_STEP5_DIR, A_STEP5_STEP, A_STEP6_DIR, A_STEP6_STEP, B_STEP5_DIR, B_STEP5_STEP, B_STEP6_DIR, B_STEP6_STEP, STEP5_DIR, STEP5_STEP, STEP6_DIR, STEP6_STEP
Changed lines of the file:
@@
 $EndComp
 Text Label 8500 5100 0    50   ~ 0
-STEP5_DIR
+BRAKE1_DIR
 Text Label 8500 5400 0    50   ~ 0
-STEP5_STEP
+BRAKE1_STEP
 $Comp
 L +5V #PWR?
@@
 $EndComp
 Text Label 10140 5500 0    50   ~ 0
-STEP6_DIR
+BRAKE2_DIR
 Text Label 10150 5200 0    50   ~ 0
-STEP6_STEP
+BRAKE2_STEP
 $Comp
 L GNDD #PWR?
@@
 B_STEP4_STEP
 Text Label 8500 4900 0    50   ~ 0
-A_STEP5_DIR
+A_BRAKE1_DIR
 Text Label 8500 5000 0    50   ~ 0
-B_STEP5_DIR
+B_BRAKE1_DIR
 Text Label 8500 5200 0    50   ~ 0
-A_STEP5_STEP
+A_BRAKE1_STEP
 Text Label 8500 5300 0    50   ~ 0
-B_STEP5_STEP
+B_BRAKE1_STEP
 Text Label 10140 5300 0    50   ~ 0
-A_STEP6_DIR
+A_BRAKE2_DIR
 Text Label 10140 5400 0    50   ~ 0
-B_STEP6_DIR
+B_BRAKE2_DIR
 Text Label 10130 5000 0    50   ~ 0
-A_STEP6_STEP
+A_BRAKE2_STEP
 Text Label 10130 5100 0    50   ~ 0
-B_STEP6_STEP
+B_BRAKE2_STEP
 Text Label 7560 1950 0    50   ~ 0
 A_STEP1_DIR
@@
 A_STEP4_STEP
 Text Label 7570 2250 0    50   ~ 0
-A_STEP5_DIR
+A_BRAKE1_DIR
 Text Label 7560 2550 0    50   ~ 0
-A_STEP5_STEP
+A_BRAKE1_STEP
 Text Label 7560 2650 0    50   ~ 0
-A_STEP6_DIR
+A_BRAKE2_DIR
 Text Label 7560 2750 0    50   ~ 0
-A_STEP6_STEP
+A_BRAKE2_STEP
 $Comp
 L GNDD #PWR?
@@
 B_STEP4_STEP
 Text Label 4080 3520 0    50   ~ 0
-B_STEP5_DIR
+B_BRAKE1_DIR
 Text Label 4070 3820 0    50   ~ 0
-B_STEP5_STEP
+B_BRAKE1_STEP
 Text Label 4070 3920 0    50   ~ 0
-B_STEP6_DIR
+B_BRAKE2_DIR
 Text Label 4070 4020 0    50   ~ 0
-B_STEP6_STEP
+B_BRAKE2_STEP
 $Comp
 L TPS3813 U?
