File: StepperNode_Brake_Failsafe.sch (KiCad schematic (older format))
At the start: 9 parts

Commit message: First Revision -
Parts:
- removed D?: 1N4004, symbol D
- removed P? (x2): CONN_01X02_2XMNT, symbol CONN_01X02_2XMNT
- removed RL?: TQ2-5V, symbol TQ2-5V
- added D1: BAS16,215, RLOOP_FOOTPRINTS:rLoop_SOT23, symbol BAS16,215
- added P6: TE_640456-8, RLOOP_FOOTPRINTS:rLoop_TE640456-8, symbol TE_640456-8
- added RL1: TQ2-5V, RLOOP_FOOTPRINTS:rLoop_DIP10, symbol TQ2-5V
- gave numbers to parts that had none: 5
Connections:
- net at U15.3 (DRAIN): now also D1.1 (A), RL1.10
- new net: P6.1 (P1), RL1.3
- new net: P6.2 (P2), RL1.4
- new net: P6.5 (P5), RL1.7
- new net: P6.4 (P4), RL1.8
- new net +5V: D1.3 (K), RL1.1
- no-connect marks 0 -> 1
Other:
- note added: "The purpose of this function is to ensure that if the WDT_GOOD signal \ngoes low the drive controllers do not drop out if the interlock is enabled.\n"
- note removed: "The purpose of this function is to:\n1. Ensure that if the WDT_GOOD signal goes low the drive controllers do not drop out if the interlock is enabled.\n2. Loss of either 24VA or 24VB will not cause the loss of an individual drive controller."
Changed lines of the file:
@@
 Text Notes 11950 10500 0    60   ~ 0
 Original Author: SafetyLok
-$Comp
-L CONN_01X02_2XMNT P?
-U 1 1 575559F0
-P 12350 4250
-F 0 "P?" H 12350 4400 50  0000 C CNN
-F 1 "CONN_01X02_2XMNT" V 12450 4250 50  0000 C CNN
-F 2 "" H 12350 4250 50  0000 C CNN
-F 3 "" H 12350 4250 50  0000 C CNN
-	1    12350 4250
-	1    0    0    -1
-$EndComp
 Text Notes 12700 4250 0    60   ~ 0
 Brake 1 G210x\nEnable Link
@@
 Text HLabel 5650 4150 0    60   Input ~ 0
 WDT_GOOD
-$Comp
-L CONN_01X02_2XMNT P?
-U 1 1 5753DAA1
-P 12300 5350
-F 0 "P?" H 12300 5500 50  0000 C CNN
-F 1 "CONN_01X02_2XMNT" V 12400 5350 50  0000 C CNN
-F 2 "" H 12300 5350 50  0000 C CNN
-F 3 "" H 12300 5350 50  0000 C CNN
-	1    12300 5350
-	1    0    0    -1
-$EndComp
-Text Notes 12650 5350 0    60   ~ 0
+Text Notes 12750 4650 0    60   ~ 0
 Brake 2 G210x\nEnable Link
 Text HLabel 4150 5400 0    60   Input ~ 0
@@
 	9050 4550 9050 4900
 $Comp
-L GNDD #PWR?
+L GNDD #PWR100
 U 1 1 575D769D
 P 9050 5900
-F 0 "#PWR?" H 9050 5650 50  0001 C CNN
+F 0 "#PWR100" H 9050 5650 50  0001 C CNN
 F 1 "GNDD" H 9050 5750 50  0000 C CNN
 F 2 "" H 9050 5900 50  0000 C CNN
@@
 	1    0    0    -1
 $EndComp
-$Comp
-L D D?
-U 1 1 575D7CC9
-P 8750 4350
-F 0 "D?" H 8750 4450 50  0000 C CNN
-F 1 "1N4004" H 8750 4250 50  0000 C CNN
-F 2 "" H 8750 4350 50  0000 C CNN
-F 3 "" H 8750 4350 50  0000 C CNN
-	1    8750 4350
-	0    1    1    0
-$EndComp
 Wire Wire Line
 	8750 4150 9050 4150
@@
 Wire Wire Line
 	8750 4550 8750 4500
-Text Notes 3800 1650 0    60   ~ 0
-The purpose of this function is to:\n1. Ensure that if the WDT_GOOD signal goes low the drive controllers do not drop out if the interlock is enabled.\n2. Loss of either 24VA or 24VB will not cause the loss of an individual drive controller.
-Wire Wire Line
-	10250 4550 11250 4550
-Wire Wire Line
-	11250 4550 11250 5300
-Wire Wire Line
-	11250 5300 12100 5300
-Wire Wire Line
-	10250 4650 11150 4650
-Wire Wire Line
-	11150 4650 11150 5400
-Wire Wire Line
-	11150 5400 12100 5400
+Wire Wire Line
+	10250 4550 11300 4550
+Wire Wire Line
+	10250 4650 11350 4650
 Wire Wire Line
 	5000 5400 4150 5400
@@
 	4150 5600 5000 5600
 $Comp
-L GNDD #PWR?
+L GNDD #PWR94
 U 1 1 575DA88C
 P 5500 6000
-F 0 "#PWR?" H 5500 5750 50  0001 C CNN
+F 0 "#PWR94" H 5500 5750 50  0001 C CNN
 F 1 "GNDD" H 5500 5850 50  0000 C CNN
 F 2 "" H 5500 6000 50  0000 C CNN
@@
 Output is high when either\nInterlock is on
 $Comp
-L GNDD #PWR?
+L GNDD #PWR96
 U 1 1 575DAC78
 P 7200 5900
-F 0 "#PWR?" H 7200 5650 50  0001 C CNN
+F 0 "#PWR96" H 7200 5650 50  0001 C CNN
 F 1 "GNDD" H 7200 5750 50  0000 C CNN
 F 2 "" H 7200 5900 50  0000 C CNN
@@
 Text Notes 7000 6500 0    60   ~ 0
 If WDT or any Interlock is active then\nThe drive controllers always remain active.\nIn this mode a WDT fault can't cause loss of drive motors.
-Text Notes 9000 3900 1    60   ~ 0
+Text Notes 8450 3950 1    60   ~ 0
 Todo:\nPower RLY from redundant source.
 $Comp
-L NUD3124LT1G U?
+L NUD3124LT1G U15
 U 1 1 575A7BBF
 P 8750 5100
-F 0 "U?" H 8750 5200 60  0000 C CNN
+F 0 "U15" H 8750 5200 60  0000 C CNN
 F 1 "NUD3124LT1G" H 9450 4450 60  0000 C CNN
 F 2 "RLOOP_FOOTPRINTS:rLoop_SOT23" H 8650 5100 60  0001 C CNN
@@
 $EndComp
 $Comp
-L 74LVC1G32GW,125 U?
+L 74LVC1G32GW,125 U13
 U 1 1 575A8256
 P 5200 5250
-F 0 "U?" H 5200 5400 60  0000 C CNN
+F 0 "U13" H 5200 5400 60  0000 C CNN
 F 1 "74LVC1G32GW,125" H 6000 4600 60  0000 C CNN
 F 2 "RLOOP_FOOTPRINTS:rLoop_SOT353" H 5100 5300 60  0001 C CNN
@@
 $EndComp
 $Comp
-L +3V3_A #PWR?
+L +3V3_A #PWR93
 U 1 1 575A85D8
 P 5500 5050
-F 0 "#PWR?" H 5500 4900 50  0001 C CNN
+F 0 "#PWR93" H 5500 4900 50  0001 C CNN
 F 1 "+3V3_A" H 5500 5190 50  0000 C CNN
 F 2 "" H 5500 5050 60  0000 C CNN
@@
 $EndComp
 $Comp
-L +3V3_A #PWR?
+L +3V3_A #PWR95
 U 1 1 575A85F8
 P 7200 4950
-F 0 "#PWR?" H 7200 4800 50  0001 C CNN
+F 0 "#PWR95" H 7200 4800 50  0001 C CNN
 F 1 "+3V3_A" H 7200 5090 50  0000 C CNN
 F 2 "" H 7200 4950 60  0000 C CNN
@@
 $EndComp
 $Comp
-L C_100nF_50V C?
+L C_100nF_50V C24
 U 1 1 575A8625
 P 5450 7000
-F 0 "C?" H 5475 7100 50  0000 L CNN
+F 0 "C24" H 5475 7100 50  0000 L CNN
 F 1 "C_100nF_50V" H 5475 6900 50  0000 L CNN
 F 2 "RLOOP_FOOTPRINTS:rLoop_C_0603" H 5488 6850 50  0001 C CNN
@@
 $EndComp
 $Comp
-L GNDD #PWR?
+L GNDD #PWR92
 U 1 1 575A86D0
 P 5450 7150
-F 0 "#PWR?" H 5450 6900 50  0001 C CNN
+F 0 "#PWR92" H 5450 6900 50  0001 C CNN
 F 1 "GNDD" H 5450 7000 50  0000 C CNN
 F 2 "" H 5450 7150 50  0000 C CNN
@@
 $EndComp
 $Comp
-L +3V3_A #PWR?
+L +3V3_A #PWR91
 U 1 1 575A86E0
 P 5450 6850
-F 0 "#PWR?" H 5450 6700 50  0001 C CNN
+F 0 "#PWR91" H 5450 6700 50  0001 C CNN
 F 1 "+3V3_A" H 5450 6990 50  0000 C CNN
 F 2 "" H 5450 6850 60  0000 C CNN
@@
 $EndComp
 $Comp
-L C_100nF_50V C?
+L C_100nF_50V C25
 U 1 1 575A891A
 P 7200 7050
-F 0 "C?" H 7225 7150 50  0000 L CNN
+F 0 "C25" H 7225 7150 50  0000 L CNN
 F 1 "C_100nF_50V" H 7225 6950 50  0000 L CNN
 F 2 "RLOOP_FOOTPRINTS:rLoop_C_0603" H 7238 6900 50  0001 C CNN
@@
 $EndComp
 $Comp
-L GNDD #PWR?
+L GNDD #PWR98
 U 1 1 575A8920
 P 7200 7200
-F 0 "#PWR?" H 7200 6950 50  0001 C CNN
+F 0 "#PWR98" H 7200 6950 50  0001 C CNN
 F 1 "GNDD" H 7200 7050 50  0000 C CNN
 F 2 "" H 7200 7200 50  0000 C CNN
@@
 $EndComp
 $Comp
-L +3V3_A #PWR?
+L +3V3_A #PWR97
 U 1 1 575A8926
 P 7200 6900
-F 0 "#PWR?" H 7200 6750 50  0001 C CNN
+F 0 "#PWR97" H 7200 6750 50  0001 C CNN
 F 1 "+3V3_A" H 7200 7040 50  0000 C CNN
 F 2 "" H 7200 6900 60  0000 C CNN
@@
 $EndComp
 $Comp
-L 74LVC1G32GW,125 U?
+L 74LVC1G32GW,125 U14
 U 1 1 575A8AA1
 P 6900 5150
-F 0 "U?" H 6900 5300 60  0000 C CNN
+F 0 "U14" H 6900 5300 60  0000 C CNN
 F 1 "74LVC1G32GW,125" H 7700 4500 60  0000 C CNN
 F 2 "RLOOP_FOOTPRINTS:rLoop_SOT353" H 6800 5200 60  0001 C CNN
@@
 	1    0    0    -1
 $EndComp
-$Comp
-L TQ2-5V RL?
-U 1 1 575A2812
+NoConn ~ 9500 4400
+$Comp
+L TQ2-5V RL1
+U 1 1 57653444
 P 9250 4000
-F 0 "RL?" H 9650 4050 60  0000 C CNN
+F 0 "RL1" H 9650 4050 60  0000 C CNN
 F 1 "TQ2-5V" H 9650 3200 60  0000 C CNN
-F 2 "" H 9250 3250 60  0000 C CNN
+F 2 "RLOOP_FOOTPRINTS:rLoop_DIP10" H 9250 3250 60  0001 C CNN
 F 3 "" H 9250 3250 60  0000 C CNN
 	1    9250 4000
 	1    0    0    -1
 $EndComp
+$Comp
+L +5V_A #PWR99
+U 1 1 5765374C
+P 8750 4150
+F 0 "#PWR99" H 8750 4000 50  0001 C CNN
+F 1 "+5V_A" H 8750 4290 50  0000 C CNN
+F 2 "" H 8750 4150 60  0000 C CNN
+F 3 "" H 8750 4150 60  0000 C CNN
+	1    8750 4150
+	1    0    0    -1
+$EndComp
+$Comp
+L BAS16,215 D1
+U 1 1 5765377B
+P 8750 4350
+F 0 "D1" H 8750 4450 50  0000 C CNN
+F 1 "BAS16,215" H 8750 4250 50  0000 C CNN
+F 2 "RLOOP_FOOTPRINTS:rLoop_SOT23" H 8650 4350 50  0001 C CNN
+F 3 "" H 8750 4350 50  0000 C CNN
+	1    8750 4350
+	0    1    1    0
+$EndComp
+$Comp
+L TE_640456-8 P6
+U 1 1 576539F1
+P 12300 4150
+F 0 "P6" H 12350 4200 50  0000 C CNN
+F 1 "TE_640456-8" V 12450 3750 50  0000 C CNN
+F 2 "RLOOP_FOOTPRINTS:rLoop_TE640456-8" H 12350 3750 50  0001 C CNN
+F 3 "" H 12350 3750 50  0000 C CNN
+	1    12300 4150
+	1    0    0    -1
+$EndComp
+Wire Wire Line
+	11300 4550 11300 4500
+Wire Wire Line
+	11300 4500 12150 4500
+Wire Wire Line
+	11350 4650 11350 4600
+Wire Wire Line
+	11350 4600 12150 4600
+Text Notes 2850 3300 0    60   ~ 0
+The purpose of this function is to ensure that if the WDT_GOOD signal \ngoes low the drive controllers do not drop out if the interlock is enabled.\n
 $EndSCHEMATC
