File: StepperNode_DAC_A.sch (KiCad schematic (older format))
At the start: 9 parts

Commit message: Remove Gimbal Functions
Connections:
- net labels removed: GIMBAL1_MLP, GIMBAL1_TEMP, GIMBAL2_MLP, GIMBAL2_TEMP, GIMBAL3_MLP, GIMBAL3_TEMP, GIMBAL4_MLP, GIMBAL4_TEMP
- wire segments 47 -> 39
Changed lines of the file:
@@
 $Descr A3 16535 11693
 encoding utf-8
-Sheet 3 17
+Sheet 17 15
 Title "DAC Channel A"
 Date ""
@@
 Wire Wire Line
 	5050 3850 6450 3850
-Wire Wire Line
-	6450 3950 5050 3950
-Wire Wire Line
-	6450 4050 5050 4050
-Text HLabel 5050 3750 0    60   Input ~ 0
-GIMBAL1_MLP
-Text HLabel 5050 3850 0    60   Input ~ 0
-GIMBAL2_MLP
-Text HLabel 5050 3950 0    60   Input ~ 0
-GIMBAL3_MLP
-Text HLabel 5050 4050 0    60   Input ~ 0
-GIMBAL4_MLP
 Text HLabel 5050 5250 0    60   Output ~ 0
 A_HE1_THROTTLE
@@
 Text HLabel 5050 6150 0    60   Output ~ 0
 A_AP2_THROTTLE
-Wire Wire Line
-	6450 4150 5050 4150
-Text HLabel 5050 4150 0    60   Input ~ 0
-BRAKE1_TEMP
-Wire Wire Line
-	6450 4250 5050 4250
-Text HLabel 5050 4250 0    60   Input ~ 0
+Text HLabel 5050 3850 0    60   Input ~ 0
 BRAKE2_TEMP
-Wire Wire Line
-	6450 4350 5050 4350
-Text HLabel 5050 4350 0    60   Input ~ 0
-GIMBAL1_TEMP
-Wire Wire Line
-	6450 4450 5050 4450
-Text HLabel 5050 4450 0    60   Input ~ 0
-GIMBAL2_TEMP
-Wire Wire Line
-	6450 4550 5050 4550
-Text HLabel 5050 4550 0    60   Input ~ 0
-GIMBAL3_TEMP
-Wire Wire Line
-	6450 4650 5050 4650
-Text HLabel 5050 4650 0    60   Input ~ 0
-GIMBAL4_TEMP
 Wire Wire Line
 	6450 6050 5050 6050
@@
 	1    0    0    -1
 $EndComp
+Text HLabel 5050 3750 0    60   Input ~ 0
+BRAKE1_TEMP
 $EndSCHEMATC

Commit message: Update DAC's and routed gimbal position to MCU direct.
Parts:
- removed C? (x6): 0.1uF, symbol C
- removed U?: AMC7812, symbol AMC7812
- added C? (x6): C_100nF_50V, RLOOP_FOOTPRINTS:rLoop_C_0603, symbol C_100nF_50V
- added U?: AMC7812BSPAP, RLOOP_FOOTPRINTS:rLoop_PQFP64_10x10mm, symbol AMC7812BSPAP
Connections:
- net labels removed: BRAKE1_MLP, BRAKE2_MLP
- wire segments 39 -> 37
Changed lines of the file:
@@
 $Descr A3 16535 11693
 encoding utf-8
-Sheet 17 15
+Sheet 14 15
 Title "DAC Channel A"
 Date ""
@@
 Text Notes 11950 10500 0    60   ~ 0
 Original Author: SafetyLok
-$Comp
-L AMC7812 U?
-U 1 1 57505A3B
-P 6650 6800
-F 0 "U?" H 8900 11050 60  0000 C CNN
-F 1 "AMC7812" H 8750 6750 60  0000 C CNN
-F 2 "" H 7950 9500 60  0000 C CNN
-F 3 "" H 7950 9500 60  0000 C CNN
-	1    6650 6800
-	1    0    0    -1
-$EndComp
 Wire Wire Line
 	9150 4350 10250 4350
@@
 Wire Wire Line
 	10250 3500 9150 3500
-Text HLabel 5050 3550 0    60   Output ~ 0
-BRAKE1_MLP
-Text HLabel 5050 3650 0    60   Output ~ 0
-BRAKE2_MLP
 Wire Wire Line
 	6450 3550 5050 3550
 Wire Wire Line
 	5050 3650 6450 3650
-Wire Wire Line
-	6450 3750 5050 3750
-Wire Wire Line
-	5050 3850 6450 3850
 Text HLabel 5050 5250 0    60   Output ~ 0
 A_HE1_THROTTLE
@@
 Text HLabel 5050 6150 0    60   Output ~ 0
 A_AP2_THROTTLE
-Text HLabel 5050 3850 0    60   Input ~ 0
-BRAKE2_TEMP
 Wire Wire Line
 	6450 6050 5050 6050
@@
 Could put an LED on this for debug
 $Comp
-L C C?
-U 1 1 57564A2D
-P 5700 1350
-F 0 "C?" H 5725 1450 50  0000 L CNN
-F 1 "0.1uF" H 5725 1250 50  0000 L CNN
-F 2 "" H 5738 1200 50  0000 C CNN
-F 3 "" H 5700 1350 50  0000 C CNN
-	1    5700 1350
-	1    0    0    -1
-$EndComp
-$Comp
 L +5VA #PWR?
 U 1 1 57564A9D
@@
 $EndComp
 $Comp
-L C C?
-U 1 1 57564BD9
-P 6100 1350
-F 0 "C?" H 6125 1450 50  0000 L CNN
-F 1 "0.1uF" H 6125 1250 50  0000 L CNN
-F 2 "" H 6138 1200 50  0000 C CNN
-F 3 "" H 6100 1350 50  0000 C CNN
-	1    6100 1350
-	1    0    0    -1
-$EndComp
-$Comp
 L +5VA #PWR?
 U 1 1 57564BDF
@@
 $EndComp
 $Comp
-L C C?
-U 1 1 57564C38
-P 6450 1350
-F 0 "C?" H 6475 1450 50  0000 L CNN
-F 1 "0.1uF" H 6475 1250 50  0000 L CNN
-F 2 "" H 6488 1200 50  0000 C CNN
-F 3 "" H 6450 1350 50  0000 C CNN
-	1    6450 1350
-	1    0    0    -1
-$EndComp
-$Comp
 L +5VA #PWR?
 U 1 1 57564C3E
@@
 $EndComp
 $Comp
-L C C?
-U 1 1 57564C4A
-P 6850 1350
-F 0 "C?" H 6875 1450 50  0000 L CNN
-F 1 "0.1uF" H 6875 1250 50  0000 L CNN
-F 2 "" H 6888 1200 50  0000 C CNN
-F 3 "" H 6850 1350 50  0000 C CNN
-	1    6850 1350
-	1    0    0    -1
-$EndComp
-$Comp
 L +5VA #PWR?
 U 1 1 57564C50
@@
 $EndComp
 $Comp
-L C C?
-U 1 1 57564C9F
-P 7350 1350
-F 0 "C?" H 7375 1450 50  0000 L CNN
-F 1 "0.1uF" H 7375 1250 50  0000 L CNN
-F 2 "" H 7388 1200 50  0000 C CNN
-F 3 "" H 7350 1350 50  0000 C CNN
-	1    7350 1350
-	1    0    0    -1
-$EndComp
-$Comp
 L +3.3V #PWR?
 U 1 1 57564CBD
@@
 $EndComp
 $Comp
-L C C?
-U 1 1 57564D7D
-P 7700 1350
-F 0 "C?" H 7725 1450 50  0000 L CNN
-F 1 "0.1uF" H 7725 1250 50  0000 L CNN
-F 2 "" H 7738 1200 50  0000 C CNN
-F 3 "" H 7700 1350 50  0000 C CNN
-	1    7700 1350
-	1    0    0    -1
-$EndComp
-$Comp
 L +3.3V #PWR?
 U 1 1 57564D83
-P 7700 1200
-F 0 "#PWR?" H 7700 1050 50  0001 C CNN
-F 1 "+3.3V" H 7700 1340 50  0000 C CNN
-F 2 "" H 7700 1200 50  0000 C CNN
-F 3 "" H 7700 1200 50  0000 C CNN
-	1    7700 1200
+P 7750 1200
+F 0 "#PWR?" H 7750 1050 50  0001 C CNN
+F 1 "+3.3V" H 7750 1340 50  0000 C CNN
+F 2 "" H 7750 1200 50  0000 C CNN
+F 3 "" H 7750 1200 50  0000 C CNN
+	1    7750 1200
 	1    0    0    -1
 $EndComp
@@
 L GNDD #PWR?
 U 1 1 57564D89
-P 7700 1500
-F 0 "#PWR?" H 7700 1250 50  0001 C CNN
-F 1 "GNDD" H 7700 1350 50  0000 C CNN
-F 2 "" H 7700 1500 50  0000 C CNN
-F 3 "" H 7700 1500 50  0000 C CNN
-	1    7700 1500
-	1    0    0    -1
-$EndComp
-Text HLabel 5050 3750 0    60   Input ~ 0
+P 7750 1500
+F 0 "#PWR?" H 7750 1250 50  0001 C CNN
+F 1 "GNDD" H 7750 1350 50  0000 C CNN
+F 2 "" H 7750 1500 50  0000 C CNN
+F 3 "" H 7750 1500 50  0000 C CNN
+	1    7750 1500
+	1    0    0    -1
+$EndComp
+Text HLabel 5050 3650 0    60   Input ~ 0
+BRAKE2_TEMP
+Text HLabel 5050 3550 0    60   Input ~ 0
 BRAKE1_TEMP
+$Comp
+L C_100nF_50V C?
+U 1 1 575C98D4
+P 5700 1350
+F 0 "C?" H 5725 1450 50  0000 L CNN
+F 1 "C_100nF_50V" H 5725 1250 50  0000 L CNN
+F 2 "RLOOP_FOOTPRINTS:rLoop_C_0603" H 5738 1200 50  0001 C CNN
+F 3 "" H 5700 1350 50  0000 C CNN
+	1    5700 1350
+	1    0    0    -1
+$EndComp
+$Comp
+L C_100nF_50V C?
+U 1 1 575C9947
+P 6100 1350
+F 0 "C?" H 6125 1450 50  0000 L CNN
+F 1 "C_100nF_50V" H 6125 1250 50  0000 L CNN
+F 2 "RLOOP_FOOTPRINTS:rLoop_C_0603" H 6138 1200 50  0001 C CNN
+F 3 "" H 6100 1350 50  0000 C CNN
+	1    6100 1350
+	1    0    0    -1
+$EndComp
+$Comp
+L C_100nF_50V C?
+U 1 1 575C99AA
+P 6450 1350
+F 0 "C?" H 6475 1450 50  0000 L CNN
+F 1 "C_100nF_50V" H 6475 1250 50  0000 L CNN
+F 2 "RLOOP_FOOTPRINTS:rLoop_C_0603" H 6488 1200 50  0001 C CNN
+F 3 "" H 6450 1350 50  0000 C CNN
+	1    6450 1350
+	1    0    0    -1
+$EndComp
+$Comp
+L C_100nF_50V C?
+U 1 1 575C99B0
+P 6850 1350
+F 0 "C?" H 6875 1450 50  0000 L CNN
+F 1 "C_100nF_50V" H 6875 1250 50  0000 L CNN
+F 2 "RLOOP_FOOTPRINTS:rLoop_C_0603" H 6888 1200 50  0001 C CNN
+F 3 "" H 6850 1350 50  0000 C CNN
+	1    6850 1350
+	1    0    0    -1
+$EndComp
+$Comp
+L C_100nF_50V C?
+U 1 1 575C9A29
+P 7350 1350
+F 0 "C?" H 7375 1450 50  0000 L CNN
+F 1 "C_100nF_50V" H 7375 1250 50  0000 L CNN
+F 2 "RLOOP_FOOTPRINTS:rLoop_C_0603" H 7388 1200 50  0001 C CNN
+F 3 "" H 7350 1350 50  0000 C CNN
+	1    7350 1350
+	1    0    0    -1
+$EndComp
+$Comp
+L C_100nF_50V C?
+U 1 1 575C9A2F
+P 7750 1350
+F 0 "C?" H 7775 1450 50  0000 L CNN
+F 1 "C_100nF_50V" H 7775 1250 50  0000 L CNN
+F 2 "RLOOP_FOOTPRINTS:rLoop_C_0603" H 7788 1200 50  0001 C CNN
+F 3 "" H 7750 1350 50  0000 C CNN
+	1    7750 1350
+	1    0    0    -1
+$EndComp
+$Comp
+L AMC7812BSPAP U?
+U 1 1 575CB5AF
+P 6650 2600
+F 0 "U?" H 8900 2650 60  0000 C CNN
+F 1 "AMC7812BSPAP" H 8750 -1650 60  0000 C CNN
+F 2 "RLOOP_FOOTPRINTS:rLoop_PQFP64_10x10mm" H 7950 1100 60  0001 C CNN
+F 3 "" H 7950 1100 60  0000 C CNN
+	1    6650 2600
+	1    0    0    -1
+$EndComp
 $EndSCHEMATC

Commit message: First Revision -
Parts:
- removed C?: 4.7UF, symbol C
- removed R?: 10K, symbol R
- added C46: C_4u7_25V, RLOOP_FOOTPRINTS:rLoop_C_0805, symbol C_4u7_25V
- added R19: 10K, RLOOP_FOOTPRINTS:rLoop_R_0603, symbol 10K
- gave numbers to parts that had none: 7
Connections:
- net labels added: +3V3_A, +5V_A
- net labels removed: +3.3V, +5VA
