File: rloopStepperNode.sch (KiCad schematic (older format))
At the start: 0 parts

Commit message: Finish isolation and add brake limit switches.
Connections:
- net labels added: BRAKE1_SW_EXT, BRAKE1_SW_RET, BRAKE2_SW_EXT, BRAKE2_SW_RET
- wire segments 149 -> 160
Changed lines of the file:
@@
 F9 "CHA_BRAKE2_DIR" I L 14300 4800 60
 F10 "CHB_BRAKE2_STEP" I L 14300 6300 60
+F11 "BRAKE1_SW_RET" O L 14300 5200 60
+F12 "BRAKE1_SW_EXT" O L 14300 5300 60
+F13 "BRAKE2_SW_RET" O L 14300 5400 60
+F14 "BRAKE2_SW_EXT" O L 14300 5500 60
 $EndSheet
 $Sheet
@@
 F25 "IB_FR_TX" O R 2100 3600 60
 F26 "IB_FR_RX_3V" I R 2100 3700 60
+F27 "BRAKE1_SW_EXT" I R 2100 4050 60
+F28 "BRAKE1_SW_RET" I R 2100 4150 60
+F29 "BRAKE2_SW_EXT" I R 2100 4250 60
+F30 "BRAKE2_SW_RET" I R 2100 4350 60
 $EndSheet
 $Sheet
@@
 Text Label 7400 2450 0    60   ~ 0
 BRAKE2_MLP_3V
-Wire Wire Line
-	5500 5550 6400 5550
-Text Label 5550 5550 0    60   ~ 0
-STEP_DIR_CTRL
 Wire Wire Line
 	5650 6300 6550 6300
@@
 F25 "IB_FR_TX" O R 2100 8750 60
 F26 "IB_FR_RX_3V" I R 2100 8850 60
+F27 "BRAKE1_SW_EXT" I R 2100 9200 60
+F28 "BRAKE1_SW_RET" I R 2100 9300 60
+F29 "BRAKE2_SW_EXT" I R 2100 9400 60
+F30 "BRAKE2_SW_RET" I R 2100 9500 60
 $EndSheet
 Wire Wire Line
@@
 Text Label 2250 7100 0    60   ~ 0
 BRAKE2_MLP_3V
+Wire Wire Line
+	14300 5200 13300 5200
+Text Label 13450 5200 0    60   ~ 0
+BRAKE1_SW_RET
+Wire Wire Line
+	14300 5300 13300 5300
+Text Label 13450 5300 0    60   ~ 0
+BRAKE1_SW_EXT
+Wire Wire Line
+	14300 5400 13300 5400
+Text Label 13450 5400 0    60   ~ 0
+BRAKE2_SW_RET
+Wire Wire Line
+	14300 5500 13300 5500
+Text Label 13450 5500 0    60   ~ 0
+BRAKE2_SW_EXT
+Wire Wire Line
+	3100 4050 2100 4050
+Text Label 2250 4150 0    60   ~ 0
+BRAKE1_SW_RET
+Wire Wire Line
+	3100 4150 2100 4150
+Text Label 2250 4050 0    60   ~ 0
+BRAKE1_SW_EXT
+Wire Wire Line
+	3100 4250 2100 4250
+Text Label 2250 4350 0    60   ~ 0
+BRAKE2_SW_RET
+Wire Wire Line
+	3100 4350 2100 4350
+Text Label 2250 4250 0    60   ~ 0
+BRAKE2_SW_EXT
+Wire Wire Line
+	3100 9200 2100 9200
+Text Label 2250 9300 0    60   ~ 0
+BRAKE1_SW_RET
+Wire Wire Line
+	3100 9300 2100 9300
+Text Label 2250 9200 0    60   ~ 0
+BRAKE1_SW_EXT
+Wire Wire Line
+	3100 9400 2100 9400
+Text Label 2250 9500 0    60   ~ 0
+BRAKE2_SW_RET
+Wire Wire Line
+	3100 9500 2100 9500
+Text Label 2250 9400 0    60   ~ 0
+BRAKE2_SW_EXT
 $EndSCHEMATC
